Commit message: add map_nav same time file

File: src/nav_demo/urdf/car.urdf.xacro (robot description, xacro)
@@ -7,3 +7,4 @@
     <xacro:include filename="sensor/sensor_laser.urdf.xacro" />
     <xacro:include filename="sensor/sensor_motion.urdf.xacro" />
+    <xacro:include filename="sensor/depth_camera.urdf.xacro" />
 </robot>

File: src/nav_demo/urdf/laser.urdf.xacro (robot description, xacro)
@@ -36,4 +36,24 @@
         <material>Gazebo/White</material>
     </gazebo>
+    <!-- 固定
+    <link name="fixed_point1">
+      <visual>
+        <geometry>
+          <sphere radius="0.001" />
+        </geometry>
+      </visual>
+    </link>
+    <link name="fixed_point2">
+      <visual>
+        <geometry>
+          <sphere radius="0.001" />
+        </geometry>
+      </visual>
+    </link>
+    <joint name="fixed_points_link" type="fixed">
+        <parent link="fixed_point1" />
+        <child link="fixed_point2" />
+        <origin xyz="${support_x} ${support_y} ${support_z}" />
+    </joint> -->
     <!-- 雷达属性 -->
     <xacro:property name="laser_length" value="0.05" /> <!-- 雷达长度 -->
